File: pcb/LEFT/multiboard_LEFT/multiboard_LEFT.kicad_pcb (KiCad board)
At the start: 2 copper layers, 109 parts, among them SW10 SW_Push, SW11 SW_Push, SW12 SW_Push, SW13 SW_Push, SW14 SW_Push, SW15 SW_Push, SW16 SW_Push, SW17 SW_Push, SW18 SW_Push, SW19 SW_Push, SW20 SW_Push, SW21 SW_Push, SW22 SW_Push, SW23 SW_Push, SW24 SW_Push, SW25 SW_Push, SW26 SW_Push, SW27 SW_Push, SW28 SW_Push, SW29 SW_Push, SW3 SW_Push, SW30 SW_Push, SW31 SW_Push, SW32 SW_Push, SW33 SW_Push, SW34 SW_Push, SW35 SW_Push, SW36 SW_Push, SW37 SW_Push, SW38 SW_Push, SW39 SW_Push, SW4 SW_Push, SW40 SW_Push, SW41 SW_Push, SW42 SW_Push, SW46 SW_Push, SW47 SW_Push, SW48 SW_Push, SW49 SW_Push, SW5 SW_Push, SW50 SW_Push, SW51 SW_Push, SW52 SW_Push, SW56 SW_Push, SW57 SW_Push, SW58 SW_Push, SW59 SW_Push, SW6 SW_Push, SW60 SW_Push, SW61 SW_Push, SW62 SW_Push, SW7 SW_Push, SW8 SW_Push, SW9 SW_Push, U1 ESP32-S3-DEVKITC-1-N8R2

Commit message: finishing LEFT PCB
Parts:
- added SW1: RotaryEncoder_Switch, Rotary_Encoder:RotaryEncoder_Alps_EC11E-Switch_Vertical_H20mm_CircularMountingHoles, F.Cu at (52.2, 39.2)
- added SW2: RotaryEncoder_Switch, Rotary_Encoder:RotaryEncoder_Alps_EC11E-Switch_Vertical_H20mm_CircularMountingHoles, F.Cu at (82.2, 39.2)
- D1, D10, D11, D12, D13, D14, D15, D16, D17, D18, D19, D2, D20, D21, D22, D23, D24, D25, D26, D27, D28, D29, D3, D30, D31, D32, D33, D34, D35, D36, D37, D38, D39, D4, D40, D44, D45, D46, D47, D48, D49, D5, D50, D54, D55, D56, D57, D58, D59, D6, D60, D7, D8, D9, SW10, SW11, SW12, SW13, SW14, SW15, SW16, SW17, SW18, SW19, SW20, SW21, SW22, SW23, SW24, SW25, SW26, SW27, SW28, SW29, SW3, SW30, SW31, SW32, SW33, SW34, SW35, SW36, SW37, SW38, SW39, SW4, SW40, SW41, SW42, SW46, SW47, SW48, SW49, SW5, SW50, SW51, SW52, SW56, SW57, SW58, SW59, SW6, SW60, SW61, SW62, SW7, SW8, SW9: moved to B.Cu
- moved SW12 181.4 mm to (232.8, 142.3), turned to 165 degrees
- moved SW22 168.5 mm to (238.0, 123.1), turned to 165 degrees
- moved SW11 163.7 mm to (213.5, 137.7), turned to 168 degrees
- moved SW32 155.8 mm to (243.2, 103.7), turned to 165 degrees
- moved SW62 150.5 mm to (258.6, 46.3), turned to 165 degrees
- moved SW21 149.3 mm to (217.6, 118.2), turned to 168 degrees
- moved SW51 148.2 mm to (230.2, 59.8), turned to 168 degrees
- moved SW10 146.6 mm to (193.9, 134.0), turned to 171 degrees
- moved SW42 143.5 mm to (248.2, 84.5), turned to 165 degrees
- moved SW31 135.2 mm to (221.8, 98.6), turned to 168 degrees
- moved SW52 134.5 mm to (253.4, 65.3), turned to 165 degrees
- moved D10 134.3 mm to (231.8, 147.5), turned to -15 degrees
- moved SW20 130.7 mm to (197.0, 114.2), turned to 171 degrees
- moved SW9 130.7 mm to (174.1, 131.3), turned to 174 degrees
- moved SW61 126.9 mm to (234.4, 40.4), turned to 168 degrees
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Routing:
- net COL1: track 0.00 -> 436.0 mm, vias 0 -> 2
- net ROW1: track 0.00 -> 328.4 mm, vias 0 -> 9
- net COL2: track 0.00 -> 310.3 mm, vias 0 -> 2
- net COL3: track 0.00 -> 295.8 mm, vias 0 -> 1
- net ROW4: track 0.00 -> 286.8 mm, vias 0 -> 9
- net ROW5: track 0.00 -> 285.2 mm, vias 0 -> 10
- net COL4: track 0.00 -> 279.5 mm
- net ROW6: track 0.00 -> 271.8 mm, vias 0 -> 8
- net ROW10: track 0.00 -> 263.6 mm, vias 0 -> 7
- net ROW2: track 0.00 -> 254.7 mm, vias 0 -> 7
- net ROTB1: track 0.00 -> 249.2 mm
- net ROW3: track 0.00 -> 249.0 mm, vias 0 -> 5
- net ROTA1: track 0.00 -> 242.1 mm, vias 0 -> 2
- net BTN1: track 0.00 -> 228.5 mm
- net ROTB2: track 0.00 -> 222.0 mm, vias 0 -> 1
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- added copper zone on B.Cu, net GND
Other:
- board outline added: 234.5 x 145.5 mm

Commit message: finish left and right main pcbs
Routing:
- net ROW2: track 254.7 -> 262.5 mm
- net ROW10: track 263.6 -> 268.2 mm
- net ROW7: track 192.6 -> 196.8 mm
- net ROW5: track 285.2 -> 289.2 mm
- net COL2: track 310.3 -> 314.0 mm
- net ROW8: track 167.7 -> 169.5 mm
- net COL6: track 189.1 -> 190.8 mm
- net COL4: track 279.5 -> 280.9 mm
- net ROTA2: track 216.7 -> 216.2 mm
Other:
- board size 234.5 x 145.5 mm -> 235.3 x 146.2 mm
