File: pcb/RIGHT_Main/multiboard_RIGHT/multiboard_RIGHT.kicad_pcb (KiCad board)
At the start: 2 copper layers, 281 x 155 mm, 134 parts, among them J1 OLED, SW13 SW_Push, SW14 SW_Push, SW15 SW_Push, SW16 SW_Push, SW17 SW_Push, SW18 SW_Push, SW19 SW_Push, SW20 SW_Push, SW21 SW_Push, SW22 SW_Push, SW23 SW_Push, SW24 SW_Push, SW25 SW_Push, SW26 SW_Push, SW27 SW_Push, SW28 SW_Push, SW29 SW_Push, SW3 SW_Push, SW30 SW_Push, SW31 SW_Push, SW32 SW_Push, SW33 SW_Push, SW34 SW_Push, SW35 SW_Push, SW36 SW_Push, SW37 SW_Push, SW38 SW_Push, SW39 SW_Push, SW4 SW_Push, SW40 SW_Push, SW41 SW_Push, SW42 SW_Push, SW43 SW_Push, SW44 SW_Push, SW45 SW_Push, SW46 SW_Push, SW47 SW_Push, SW48 SW_Push, SW49 SW_Push, SW5 SW_Push, SW50 SW_Push, SW51 SW_Push, SW52 SW_Push, SW53 SW_Push, SW54 SW_Push, SW55 SW_Push, SW56 SW_Push, SW57 SW_Push, SW58 SW_Push, SW59 SW_Push, SW6 SW_Push, SW60 SW_Push, SW61 SW_Push, SW62 SW_Push, SW63 SW_Push, SW64 SW_Push, SW65 SW_Push, SW66 SW_Push, SW67 SW_Push, SW69 SW_Push, SW7 SW_Push, SW70 SW_Push, SW71 SW_Push, SW72 SW_Push, SW73 SW_Push, SW8 SW_Push, U1 ESP32-S3-DEVKITC-1-N8R2

Commit message: add headphone jack
Parts:
- added J2: PJ-320D-A, PJ:HRO_PJ-320D-A, F.Cu at (36.0, 52.4)
Connections:
- U1 pad J3_2: unconnected-(U1-U0TXD/GPIO43-PadJ3_2) -> TX
- U1 pad J3_3: unconnected-(U1-U0RXD/GPIO44-PadJ3_3) -> RX
Routing:
- net RX: track 0.00 -> 167.3 mm, vias 0 -> 3
- net TX: track 0.00 -> 108.1 mm, vias 0 -> 6
- net +3V3: track 101.9 -> 145.5 mm
- net COL4: track 347.1 -> 363.3 mm
- net ROW2: track 139.9 -> 143.4 mm
- net GND: track 0.00 -> 3.47 mm, vias 0 -> 1
- net COL2: track 370.6 -> 372.2 mm
- net COL1: track 231.6 -> 232.8 mm
